File: Radio/APRS/APRS.kicad_pcb (KiCad board)
At the start: 4 copper layers, 200 x 120 mm, 93 parts, among them J1 Filter Test, J2 Filter Test, J3 Signal, J4 Filter Test, J5 Filter Test, J6 Power, J7 I^{2}C, Q1 DMMT3904W, Q2 DMMT3904W, U1 MC1496, U2 MC1496, Y1 Crystal_Small, Y2 Crystal_Small, Y3 Crystal_Small, Y4 Crystal_Small, Y5 25MHz, Y6 Si5351A-B-GT

Commit message: Added testboards
Parts:
- removed AE1: Antenna_Dipole, Connector_PinHeader_2.54mm:PinHeader_1x02_P2.54mm_Vertical
- removed C16: 50p, Capacitor_SMD:C_0603_1608Metric_Pad1.08x0.95mm_HandSolder
- removed C18, C20: 10n, Capacitor_SMD:C_0603_1608Metric_Pad1.08x0.95mm_HandSolder
- removed C29, C31: 10nF, Capacitor_SMD:C_0603_1608Metric_Pad1.08x0.95mm_HandSolder
- removed J4: Filter Test, Connector_Coaxial:SMA_Molex_73251-1153_EdgeMount_Horizontal
- removed L5: 1.2uH, radio:Inductor_P15.24mm_Horizontal
- removed Q2: DMMT3904W, Package_TO_SOT_SMD:SOT-363_SC-70-6
- removed R26: 8.3k, Resistor_SMD:R_0603_1608Metric_Pad0.98x0.95mm_HandSolder
- removed R28: 2.2k, Resistor_SMD:R_0603_1608Metric_Pad0.98x0.95mm_HandSolder
- removed R30: 50, Resistor_SMD:R_0603_1608Metric_Pad0.98x0.95mm_HandSolder
- removed R32: 1k, Resistor_SMD:R_0603_1608Metric_Pad0.98x0.95mm_HandSolder
- removed R34: 6, Resistor_SMD:R_0603_1608Metric_Pad0.98x0.95mm_HandSolder
- added C33: 10nF, Capacitor_SMD:C_0603_1608Metric_Pad1.08x0.95mm_HandSolder, F.Cu at (116.1, 88.2)
- added C34: 10nF, Capacitor_SMD:C_0603_1608Metric_Pad1.08x0.95mm_HandSolder, F.Cu at (141.8, 110.9)
- added J8: Antenna Output, Connector_Coaxial:SMA_Molex_73251-1153_EdgeMount_Horizontal, F.Cu at (127.2, 164.1)
- C15: value 50p -> 50pF
- C17, C19: value 10n -> 10nF
- R24: value 22k -> 0
- moved L4 202.7 mm to (111.3, 142.6)
- moved C30 197.6 mm to (110.5, 139.3)
- moved C15 186.4 mm to (127.2, 158.7), turned to -90 degrees
- moved R33 167.5 mm to (138.5, 150.7)
- moved R25 163.2 mm to (138.1, 153.6)
- moved Q1 159.9 mm to (128.0, 148.3)
- moved R31 158.8 mm to (138.5, 148.2), turned to 0 degrees
- moved J5 157.8 mm to (161.4, 164.2), turned to 90 degrees
- moved R24 134.0 mm to (161.5, 156.4), turned to 0 degrees
- moved C12 125.0 mm to (127.7, 124.5), turned to 0 degrees
- moved C24 123.2 mm to (171.4, 119.9), turned to 0 degrees
- moved C3 123.1 mm to (146.8, 104.4), turned to 180 degrees
- moved R16 122.4 mm to (133.7, 124.5), turned to 0 degrees
- moved J6 121.7 mm to (178.9, 118.3)
- moved R6 120.3 mm to (146.8, 102.4), turned to 0 degrees
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Connections:
- C15 pad 1: Net-(Q2A-C1) -> Net-(Q1B-C2)
- C19 pad 2: Net-(Q2A-B1) -> Net-(Q1B-B2)
- J5 pad 1: /OUT_{MIXER+} -> Net-(J5-In)
- L4 pad 2: Net-(Q2A-C1) -> Net-(Q1B-C2)
- Q1 pad 3: VCC -> Net-(Q1B-C2)
- Q1 pad 4: /PA- -> Net-(Q1B-E2)
- R24 pad 1: VCC -> /OUT_{MIXER+}
- R24 pad 2: Net-(Q1B-B2) -> Net-(J5-In)
- R25 pad 2: Net-(Q2A-B1) -> Net-(Q1B-B2)
- R31 pad 1: Net-(Q2A-B1) -> Net-(Q1B-B2)
- R33 pad 1: Net-(Q2A-E1) -> Net-(Q1B-E2)
Routing:
- net Net-(Q2B-C2): track 26.7 -> 0.00 mm
- net /OUT_{MIXER+}: track 43.3 -> 18.3 mm
- net /LO_{2}: track 30.1 -> 5.21 mm
- net /OUT_{MIXER-}: track 35.2 -> 10.9 mm
- net Net-(Q1B-C2): track 0.00 -> 15.9 mm
- net Net-(U2-IN+): track 25.2 -> 9.38 mm
- net Net-(Q1A-B1): track 13.4 -> 0.00 mm
- net Net-(Q2A-C1): track 13.2 -> 0.00 mm
- net VCC: track 32.0 -> 19.8 mm, vias 17 -> 21
- net Net-(Q2B-B2): track 11.5 -> 0.00 mm
- net Net-(Q2A-B1): track 11.4 -> 0.00 mm
- net Net-(Q1B-B2): track 11.3 -> 0.00 mm
- net GND: track 37.3 -> 27.8 mm, vias 151 -> 161
- net /PA-: track 7.54 -> 0.00 mm
- net /PA+: track 7.44 -> 0.00 mm
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