File: Radio/APRS/APRS.kicad_sch (KiCad schematic)
At the start: 93 parts, among them J1 Filter Test, J2 Filter Test, J3 Signal, J4 Filter Test, J5 Filter Test, J6 Power, J7 I^{2}C, Q1 DMMT3904W, Q2 DMMT3904W, U1 MC1496, U2 MC1496, Y1 Crystal_Small, Y2 Crystal_Small, Y3 Crystal_Small, Y4 Crystal_Small, Y5 25MHz, Y6 Si5351A-B-GT

Commit message: Added testboards
Parts:
- removed AE1: Antenna_Dipole, Connector_PinHeader_2.54mm:PinHeader_1x02_P2.54mm_Vertical, symbol Device:Antenna_Dipole
- removed C16: 50pF, Capacitor_SMD:C_0603_1608Metric_Pad1.08x0.95mm_HandSolder, symbol Device:C_Small
- removed C18, C20, C29, C31: 10nF, Capacitor_SMD:C_0603_1608Metric_Pad1.08x0.95mm_HandSolder, symbol Device:C_Small
- removed J4: Filter Test, Connector_Coaxial:SMA_Molex_73251-1153_EdgeMount_Horizontal, symbol Connector:Conn_Coaxial_Small
- removed L5: 1.2uH, radio:Inductor_P15.24mm_Horizontal, symbol Device:L_Small
- removed Q2: DMMT3904W, Package_TO_SOT_SMD:SOT-363_SC-70-6, symbol radio:DMMT3904W
- removed R26: 8.3k, Resistor_SMD:R_0603_1608Metric_Pad0.98x0.95mm_HandSolder, symbol Device:R_Small
- removed R28: 2.2k, Resistor_SMD:R_0603_1608Metric_Pad0.98x0.95mm_HandSolder, symbol Device:R_Small
- removed R30: 50, Resistor_SMD:R_0603_1608Metric_Pad0.98x0.95mm_HandSolder, symbol Device:R_Small
- removed R32: 1k, Resistor_SMD:R_0603_1608Metric_Pad0.98x0.95mm_HandSolder, symbol Device:R_Small
- removed R34: 6, Resistor_SMD:R_0603_1608Metric_Pad0.98x0.95mm_HandSolder, symbol Device:R_Small
- added C33, C34: 10nF, Capacitor_SMD:C_0603_1608Metric_Pad1.08x0.95mm_HandSolder, symbol Device:C_Small
- added J8: Antenna Output, Connector_Coaxial:SMA_Molex_73251-1153_EdgeMount_Horizontal, symbol Connector:Conn_Coaxial_Small
- R24: value 22k -> 0
Connections:
- net PA- is gone; now on an unnamed net: Q1.4 (E2)
- net GND: now also C33.2, C34.2, J8.2 (Ext)
- net OUT_{MIXER+}: now also R24.1; no longer J5.1 (In)
- net VCC: now also C33.1, C34.1; no longer Q1.3 (C2), R24.1
- net at Q1.2 (B2): now also C19.2, R25.2, R31.1; no longer R24.2
- net at C15.2: now also J8.1 (In)
- net at C15.1, L4.2: now also Q1.3 (C2)
- new net: J5.1 (In), R24.2
Other:
- note added: "Should give ~14dBm"
- note removed: "Should give ~20dBm"
- moved on the sheet: J5, Q1B
